Commit message: ic2

File: rbot/urdf/rbot.urdf (robot description, URDF)
Before this commit: robot rbot, 7 links, 6 joints
Links:
- added link Camera_base, mass 0.20962; collision mesh filename=package://rbot/meshes/Camera_base.STL; visual mesh filename=package://rbot/meshes/Camera_base.STL
- added link fan, mass 0.025691; collision mesh filename=package://rbot/meshes/fan.STL; visual mesh filename=package://rbot/meshes/fan.STL
- link Camera: mass 0.0120488103805723 -> 0.16364
- link LiDar: mass 0.0706251365392673 -> 0.2
- link base_link: mass 1.19458055963595 -> 5.4228; geometry collision mesh filename=package://rbot/meshes/base_link.STL; visual mesh filename=package://rbot/meshes/base_link.STL
- link fWheel: mass 0.0194386045440868 -> 0.34828
- link l_rWheel: mass 0.0561559686829175 -> 0.52108
- link r_rWheel: mass 0.0561559686829175 -> 0.52108
Joints:
- removed joint Camera_tc
- added joint Camera_Camera_base: type continuous, parent Camera_base, child Camera, origin xyz=0.000199999999997202 0.0644000000000001 0.0900000000000034 rpy=0 0 0, axis 0 1 0, limit effort=2.6 velocity=20
- added joint Camera_base_tc: type fixed, parent base_link, child Camera_base, origin xyz=-0.0750239674809218 -1.19645664770351E-05 0.00499999999999973 rpy=0 0 0, axis 0 0 0
- added joint fan_bc: type continuous, parent base_link, child fan, origin xyz=0.009976 -1.1899E-05 -0.069083 rpy=0 0 0, axis 0 0 -1
- joint LiDar_tc: origin xyz=0 0 0.111 rpy=0 0 0 -> xyz=-2.3967480921927E-05 -1.19645664762025E-05 0.019 rpy=0 0 0
- joint fWheel_bc: limit (none) -> effort=2.6 velocity=20; origin xyz=0.118393751374048 0 0.008 rpy=0 0 0 -> xyz=0.10498 -0.004012 -0.09452 rpy=0 0 0
- joint l_rWheel_bc: limit (none) -> effort=2.6 velocity=20; origin xyz=-0.029977 0.085216 0.013 rpy=0 0 0 -> xyz=-0.047024 0.074988 -0.08 rpy=0 0 0
- joint r_rWheel_bc: limit (none) -> effort=2.6 velocity=20; origin xyz=-0.0299768476642726 -0.0852163754058719 0.013 rpy=0 0 0 -> xyz=-0.047024 -0.094012 -0.08 rpy=0 0 0
